File: Device on Hand/Device on Hand.kicad_pcb (KiCad board)
At the start: 2 copper layers, 61 x 55.9 mm, 12 parts, among them J1 Screw_Terminal_01x02, J2 Screw_Terminal_01x02, U3 SparkFun_SEN-14480_H3LIS331DL, U4 ESP32-DEVKIT-V1

Commit message: update
Parts:
- removed U4: ESP32-DEVKIT-V1, ESP32-DEVKIT-V1:MODULE_ESP32_DEVKIT_V1
- added J3: Conn_01x15, Connector_PinSocket_2.54mm:PinSocket_1x15_P2.54mm_Vertical, F.Cu at (152.4, 91.0)
- added J4: Screw_Terminal_01x04, Connector_PinSocket_2.54mm:PinSocket_1x04_P2.54mm_Vertical, F.Cu at (157.0, 91.0)
- added U1: mini_esp32, ESP32_mini:ESP32_mini, F.Cu at (134.3, 108.3)
- moved RV2 48.9 mm to (191.8, 114.8), turned to 0 degrees
- moved RV1 48.1 mm to (191.8, 123.2), turned to 0 degrees
- moved ICL7660 45.8 mm to (185.4, 90.8), turned to 0 degrees
- moved U3 45.2 mm to (176.5, 118.3)
- moved C3 41.6 mm to (130.1, 135.9)
- moved C2 40.7 mm to (122.4, 135.9)
- moved J1 39.9 mm to (175.1, 95.0), turned to 0 degrees
- moved J2 28.7 mm to (162.9, 95.0), turned to 0 degrees
- moved MCP6002 27.2 mm to (151.7, 130.9), turned to 0 degrees
- moved R1 19.9 mm to (156.9, 102.4), turned to 0 degrees
- moved C1 19.5 mm to (163.2, 103.5)
Routing:
- net GND: track 131.8 -> 0.00 mm
- net Net-(J1-Pad1): track 84.4 -> 0.00 mm
- net Net-(C3-Pad2): track 71.6 -> 0.00 mm
- net 3.3v: track 65.7 -> 0.00 mm
- net Vout: track 62.5 -> 0.00 mm
- net MISO: track 50.7 -> 0.00 mm
- net SCL: track 50.1 -> 0.00 mm
- net MOSI: track 46.0 -> 0.00 mm
- net CS: track 40.0 -> 0.00 mm
- net 3.3Vin: track 37.0 -> 0.00 mm
- net Net-(C2-Pad2): track 32.4 -> 0.00 mm
- net Net-(C1-Pad2): track 6.82 -> 0.00 mm
- net Net-(C1-Pad1): track 6.21 -> 0.00 mm
- removed copper zone on B.Cu, net GND
- removed copper zone on F.Cu, net GND
Other:
- board outline removed
- board text removed: "100KOhms"
- board text removed: "20KOhms"
- board text removed: "ESP32-DEVKIT-V1"
- board text removed: "FORCE SENSOR"
- board text removed: "POWER SOURCE"
