File: Device on Bag/Device on Bag.kicad_pcb (KiCad board)
At the start: 2 copper layers, 50.8 x 55.9 mm, 3 parts, among them J1 Screw_Terminal_01x02, U1 Adafruit-LSM6DSO32, U2 ESP32-DEVKIT-V1

Commit message: update
Parts:
- removed U1: Adafruit-LSM6DSO32, Adafruit-LSM6DSO32:Adafruit-LSM6DSO32
- added U3: Adafruit-LSM6DSO32, Adafruit-LSM6DSO32:Adafruit-LSM6DSO32, F.Cu at (154.3, 128.3)
- U2: value ESP32-DEVKIT-V1 -> mini_esp32; footprint ESP32-DEVKIT-V1:MODULE_ESP32_DEVKIT_V1 -> ESP32_mini_KiCad_Library:ESP32_mini
- moved U2 7.35 mm to (129.5, 134.6), turned to 0 degrees
- moved J1 5.73 mm to (152.1, 150.5), turned to 90 degrees
Connections:
- J1 pad 1: Net-(J1-Pad1) -> Vin
- U2 pad 1: 3.3v -> unconnected-(U2-Pad1)
- U2 pad 12: unconnected-(U2-Pad12) -> MOSI
- U2 pad 14: unconnected-(U2-Pad14) -> SS
- U2 pad 15: MOSI -> unconnected-(U2-Pad15)
- U2 pad 16: unconnected-(U2-Pad16) -> 3.3v
- U2 pad 29: GND -> unconnected-(U2-Pad29)
- U2 pad 3: SS -> unconnected-(U2-Pad3)
- U2 pad 30: Net-(J1-Pad1) -> unconnected-(U2-Pad30)
- U2 pad 8: unconnected-(U2-Pad8) -> SCK
- U2 pad 9: SCK -> unconnected-(U2-Pad9)
Routing:
- net GND: track 71.8 -> 0.00 mm
- net 3.3v: track 41.5 -> 0.00 mm
- net Net-(J1-Pad1): track 35.9 -> 0.00 mm
- net SS: track 31.8 -> 0.00 mm
- net MISO: track 18.4 -> 0.00 mm
- net SCK: track 13.8 -> 0.00 mm
- net MOSI: track 9.40 -> 0.00 mm
Other:
- board outline removed

Commit message: update
Parts:
- added C1: 10uF, Capacitor_Tantalum_SMD:CP_EIA-3216-10_Kemet-I_Pad1.58x1.35mm_HandSolder, F.Cu at (148.0, 141.0)
- added C2: 20pF, Capacitor_SMD:C_0805_2012Metric_Pad1.18x1.45mm_HandSolder, F.Cu at (192.9, 113.2)
- added C3: 0.1uF, Capacitor_SMD:C_0805_2012Metric_Pad1.18x1.45mm_HandSolder, F.Cu at (158.2, 140.9)
- added C4: 20pF, Capacitor_SMD:C_0805_2012Metric_Pad1.18x1.45mm_HandSolder, F.Cu at (163.0, 140.9)
- added C5: 10uF, Capacitor_SMD:C_0805_2012Metric_Pad1.18x1.45mm_HandSolder, F.Cu at (153.4, 140.9)
- added D1: BLUE LED, LED_SMD:LED_0805_2012Metric_Pad1.15x1.40mm_HandSolder, F.Cu at (168.1, 140.8)
- added D2: RED LED, LED_SMD:LED_0805_2012Metric_Pad1.15x1.40mm_HandSolder, F.Cu at (184.8, 122.1)
- added D3: D_Schottky, Diode_SMD:D_SMA_Handsoldering, F.Cu at (170.7, 125.4)
- added Q1: BC847, Package_TO_SOT_SMD:SOT-23, F.Cu at (186.4, 118.3)
- added Q2: BC847, Package_TO_SOT_SMD:SOT-23, F.Cu at (177.9, 129.9)
- added R1: 10k, Resistor_SMD:R_0805_2012Metric_Pad1.20x1.40mm_HandSolder, F.Cu at (189.5, 122.0)
- added R2: 10k, Resistor_SMD:R_0805_2012Metric_Pad1.20x1.40mm_HandSolder, F.Cu at (184.7, 125.1)
- added R3: 1K, Resistor_SMD:R_0805_2012Metric_Pad1.20x1.40mm_HandSolder, F.Cu at (182.7, 128.0)
- added R4: 1K, Resistor_SMD:R_0805_2012Metric_Pad1.20x1.40mm_HandSolder, F.Cu at (192.9, 116.2)
- added R5: 10k, Resistor_SMD:R_0805_2012Metric_Pad1.20x1.40mm_HandSolder, F.Cu at (174.6, 136.3)
- added R6: 10k, Resistor_SMD:R_0805_2012Metric_Pad1.20x1.40mm_HandSolder, F.Cu at (197.7, 113.2)
- added S1: RESET, Button_Switch_SMD:SW_Push_SPST_NO_Alps_SKRK, F.Cu at (168.9, 137.1)
- added S2: BTN-0, Button_Switch_SMD:SW_Push_SPST_NO_Alps_SKRK, F.Cu at (187.2, 113.9)
- added U1: ESP32-WROOM-E, Espressif:ESP32-WROOM-32E, F.Cu at (155.3, 127.0)
- added Y1: Crystal_GND24, Crystal:Crystal_SMD_5032-4Pin_5.0x3.2mm, F.Cu at (179.0, 122.3)
- J1: value Screw_Terminal_01x02 -> USB_B_Micro; footprint TerminalBlock_Phoenix:TerminalBlock_Phoenix_MKDS-1,5-2-5.08_1x02_P5.08mm_Horizontal -> Connector_USB:USB_Micro-B_Molex-105017-0001
- U2: value mini_esp32 -> CH340G; footprint ESP32_mini_KiCad_Library:ESP32_mini -> Package_SO:SOIC-16_3.9x9.9mm_P1.27mm
- U3: value Adafruit-LSM6DSO32 -> AMS1117-3.3; footprint Adafruit-LSM6DSO32:Adafruit-LSM6DSO32 -> Package_TO_SOT_SMD:SOT-223-3_TabPin2
- moved U2 43.8 mm to (169.9, 117.4)
- moved U3 27.7 mm to (179.0, 115.8), turned to 0 degrees
- moved J1 27.1 mm to (170.6, 130.7), turned to 0 degrees
Connections:
- J1 pad 1: Vin -> VCCUSB
- J1 pad 2: GND -> Net-(J1-Pad2)
- U2 pad 1: unconnected-(U2-Pad1) -> GND
- U2 pad 10: MISO -> unconnected-(U2-Pad10)
- U2 pad 12: MOSI -> unconnected-(U2-Pad12)
- U2 pad 13: unconnected-(U2-Pad13) -> /DTR
- U2 pad 14: SS -> /RTS
- U2 pad 16: 3.3v -> Vin
- U2 pad 2: unconnected-(U2-Pad2) -> /TX0
- U2 pad 3: unconnected-(U2-Pad3) -> /RX0
- U2 pad 4: unconnected-(U2-Pad4) -> Net-(C3-Pad1)
- U2 pad 5: unconnected-(U2-Pad5) -> Net-(J1-Pad3)
- U2 pad 6: unconnected-(U2-Pad6) -> Net-(J1-Pad2)
- U2 pad 7: unconnected-(U2-Pad7) -> Net-(C2-Pad1)
- U2 pad 8: SCK -> Net-(C4-Pad1)
- U3 pad 1: unconnected-(U3-Pad1) -> GND
- U3 pad 2: unconnected-(U3-Pad2) -> +3.3V
- U3 pad 3: SS -> VCCUSB

Commit message: update
Parts:
- removed S1: RESET, Button_Switch_SMD:SW_Push_SPST_NO_Alps_SKRK
- removed S2: BTN-0, Button_Switch_SMD:SW_Push_SPST_NO_Alps_SKRK
- added SW1: RESET, Button_Switch_SMD:SW_Push_SPST_NO_Alps_SKRK, F.Cu at (164.5, 167.0)
- added SW2: FLASH, Button_Switch_SMD:SW_Push_SPST_NO_Alps_SKRK, F.Cu at (148.0, 167.0)
- C3: value 0.1uF -> 100nF
- moved R6 70.3 mm to (148.3, 163.2), turned to 180 degrees
- moved C2 57.4 mm to (154.9, 156.2)
- moved Q1 45.0 mm to (159.4, 154.3)
- moved Y1 44.2 mm to (149.2, 154.9)
- moved D2 41.8 mm to (148.0, 141.9), turned to 90 degrees
- moved R4 41.2 mm to (160.7, 141.9), turned to 90 degrees
- moved R2 41.1 mm to (159.4, 157.5)
- moved R1 40.8 mm to (164.4, 154.3), turned to 180 degrees
- moved D3 39.8 mm to (151.1, 160.0)
- moved J1 38.5 mm to (156.2, 166.4)
- moved U3 37.0 mm to (161.9, 148.6)
- moved U2 36.1 mm to (151.7, 148.6), turned to 90 degrees
- moved R3 34.5 mm to (151.1, 141.9), turned to 90 degrees
- moved Q2 31.3 mm to (164.4, 158.1), turned to 180 degrees
- moved R5 27.4 mm to (164.8, 161.9)
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Connections:
- net VCCUSB renamed VBUS
- net Vin renamed Net-(D3-Pad1)
- C1 pad 1: +3.3V -> 3.3V
- J1 pad 6: GND -> unconnected-(J1-Pad6)
- U3 pad 2: +3.3V -> 3.3V
Other:
- board outline added: 21.6 x 58.4 mm
