File: Device on Bag/Device on Bag.kicad_sch (KiCad schematic)
At the start: 4 parts, among them J1 Screw_Terminal_01x02, U1 Adafruit-LSM6DSO32, U2 ESP32-DEVKIT-V1

Commit message: update
Parts:
- removed U1: Adafruit-LSM6DSO32, Adafruit-LSM6DSO32:Adafruit-LSM6DSO32, symbol Adafruit-LSM6DSO32:Adafruit-LSM6DSO32
- removed U2: ESP32-DEVKIT-V1, ESP32-DEVKIT-V1:MODULE_ESP32_DEVKIT_V1, symbol ESP32-DEVKIT-V1:ESP32-DEVKIT-V1
- added U3: Adafruit-LSM6DSO32, Adafruit-LSM6DSO32:Adafruit-LSM6DSO32, symbol Adafruit-LSM6DSO32:Adafruit-LSM6DSO32
- U2: renamed from U?; footprint (none) -> ESP32_mini_KiCad_Library:ESP32_mini
Connections:
- net 3.3v: now also U3.6 (Vin)
- net GND: now also U3.5 (GND)
- net MISO: now also U2.10 (IO_19/D6)
- net MOSI: now also U2.12 (IO_23/D7), U3.10 (SDA)
- net SCK: now also U2.8 (IO_18/D5), U3.9 (SCL)
- net SS: now also U2.14 (IO_05/D8), U3.3 (CS)
Other:
- moved on the sheet: U2

Commit message: update
Parts:
- added J?: Conn_01x08, symbol Connector_Generic:Conn_01x08
Changed lines of the file:
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@@
     )
+  )
+  (symbol (lib_id "Connector_Generic:Conn_01x08") (at 120.65 114.935 0) (unit 1)
+    (in_bom yes) (on_board yes) (fields_autoplaced)
+    (property "Reference" "J?" (id 0) (at 123.19 114.9349 0)
+      (effects (font (size 1.27 1.27)) (justify left))
+    )
+    (property "Value" "Conn_01x08" (id 1) (at 123.19 117.4749 0)
+      (effects (font (size 1.27 1.27)) (justify left))
+    )
+    (property "Footprint" "" (id 2) (at 120.65 114.935 0)
+      (effects (font (size 1.27 1.27)) hide)
+    )
+    (property "Datasheet" "~" (id 3) (at 120.65 114.935 0)
+      (effects (font (size 1.27 1.27)) hide)
+    )
+    (pin "1")
+    (pin "2")
+    (pin "3")
+    (pin "4")
+    (pin "5")
+    (pin "6")
+    (pin "7")
+    (pin "8")
   )
   (symbol (lib_id "ESP32_mini:mini_esp32") (at 71.755 33.655 0) (unit 1)
@@
       (reference "J1") (unit 1) (value "Screw_Terminal_01x02") (footprint "TerminalBlock_Phoenix:TerminalBlock_Phoenix_MKDS-1,5-2-5.08_1x02_P5.08mm_Horizontal")
     )
+    (path "/0566322d-a8dd-4430-aedb-32e9ac72a70c"
+      (reference "J?") (unit 1) (value "Conn_01x08") (footprint "")
+    )
     (path "/115e89b3-85d3-4492-89f6-aa3c6c92c1c8"

Commit message: update
Parts:
- removed J1: Screw_Terminal_01x02, TerminalBlock_Phoenix:TerminalBlock_Phoenix_MKDS-1,5-2-5.08_1x02_P5.08mm_Horizontal, symbol Connector:Screw_Terminal_01x02
- removed J?: Conn_01x08, symbol Connector_Generic:Conn_01x08
- removed U2: mini_esp32, ESP32_mini_KiCad_Library:ESP32_mini, symbol ESP32_mini:mini_esp32
- removed U3: Adafruit-LSM6DSO32, Adafruit-LSM6DSO32:Adafruit-LSM6DSO32, symbol Adafruit-LSM6DSO32:Adafruit-LSM6DSO32
- added C1: 10uF, Capacitor_Tantalum_SMD:CP_EIA-3216-10_Kemet-I_Pad1.58x1.35mm_HandSolder, symbol Device:C_Polarized
- added C2, C4: 20pF, Capacitor_SMD:C_0805_2012Metric_Pad1.18x1.45mm_HandSolder, symbol Device:C
- added C3: 100nF, Capacitor_SMD:C_0805_2012Metric_Pad1.18x1.45mm_HandSolder, symbol Device:C
- added C5: 10uF, Capacitor_SMD:C_0805_2012Metric_Pad1.18x1.45mm_HandSolder, symbol Device:C
- added D1: BLUE LED, LED_SMD:LED_0805_2012Metric_Pad1.15x1.40mm_HandSolder, symbol Device:LED
- added D2: RED LED, LED_SMD:LED_0805_2012Metric_Pad1.15x1.40mm_HandSolder, symbol Device:LED
- added D3: D_Schottky, Diode_SMD:D_SMA_Handsoldering, symbol Device:D_Schottky
- added J1: USB_B_Micro, Connector_USB:USB_Micro-B_Molex-105017-0001, symbol Connector:USB_B_Micro
- added Q1, Q2: BC847, Package_TO_SOT_SMD:SOT-23, symbol Transistor_BJT:BC847
- added R1, R2: 10k, Resistor_SMD:R_0805_2012Metric_Pad1.20x1.40mm_HandSolder, symbol Device:R
- added R3, R4: 1K, Resistor_SMD:R_0805_2012Metric_Pad1.20x1.40mm_HandSolder, symbol Device:R
- added R5, R6: 10k, Resistor_SMD:R_0805_2012Metric_Pad1.20x1.40mm_HandSolder, symbol esp32-thing-eagle-import:10KOHM-1/10W-1%(0603)0603
- added S1: RESET, Button_Switch_SMD:SW_Push_SPST_NO_Alps_SKRK, symbol esp32-thing-eagle-import:SWITCH-MOMENTARY-2SMD-4.6X2.8MM
- added S2: FLASH, Button_Switch_SMD:SW_Push_SPST_NO_Alps_SKRK, symbol esp32-thing-eagle-import:SWITCH-MOMENTARY-2SMD-4.6X2.8MM
- added U1: ESP32-WROOM-E, Espressif:ESP32-WROOM-32E, symbol Espressif:ESP32-WROOM-E
- added U2: CH340G, Package_SO:SOIC-16_3.9x9.9mm_P1.27mm, symbol Interface_USB:CH340G
- added U3: AMS1117-3.3, Package_TO_SOT_SMD:SOT-223-3_TabPin2, symbol Regulator_Linear:AMS1117-3.3
- added Y1: Crystal_GND24, Crystal:Crystal_SMD_5032-4Pin_5.0x3.2mm, symbol Device:Crystal_GND24
Connections:
- net GND: now also C1.2, C2.2, C3.2, C4.2, C5.2, D2.1 (K), J1.5 (GND), J1.6 (Shield), R4.2, S1.1, S1.2 (1), S2.1, S2.2 (1), U1.1 (GND), U1.15 (GND), U1.38 (GND), U2.1 (GND), U3.1 (GND), Y1.2, Y1.4
- new net: Q2.1 (B), R2.2
- new net: C2.1, U2.7 (XI), Y1.1
- new net: C4.1, U2.8 (XO), Y1.3
- new net: D1.1 (K), R4.1
- new net: D3.1 (K), U2.16 (VCC)
- new net: C3.1, U2.4 (V3)
- new net: J1.3 (D+), U2.5 (UD+)
- new net: J1.2 (D-), U2.6 (UD-)
- new net: D2.2 (A), R3.2
- new net: Q1.1 (B), R1.2
- new net +3.3V: R3.1, U1.2 (3V3)
- new net 3.3V: C1.1, R5.2, R6.2, U3.2 (VO)
- new net DTR: Q2.2 (E), R1.1, U2.13 (~{DTR})
- new net EN: Q1.3 (C), R5.1, S1.3 (2), S1.4 (2), U1.3 (EN/CHIP_PU)
- new net GPIO0: Q2.3 (C), R6.1, S2.3 (2), S2.4 (2), U1.25 (GPIO0/BOOT/ADC2_CH1)
- new net GPIO2: D1.2 (A), U1.24 (ADC2_CH2/GPIO2)
- new net RTS: Q1.2 (E), R2.1, U2.14 (~{RTS})
- new net RX0: U1.34 (U0RXD/GPIO3), U2.3 (RXD)
- new net TX0: U1.35 (U0TXD/GPIO1), U2.2 (TXD)
- new net VBUS: C5.1, D3.2 (A), J1.1 (VBUS), U3.3 (VI)
Other:
- note added: "CH340G (USB-to-Serial Converter)"
- note added: "GPIO0 Button"
- note added: "Reset Button"
- note added: "Voltage Regulator"

Commit message: update
Parts:
- removed S1: RESET, Button_Switch_SMD:SW_Push_SPST_NO_Alps_SKRK, symbol esp32-thing-eagle-import:SWITCH-MOMENTARY-2SMD-4.6X2.8MM
- removed S2: FLASH, Button_Switch_SMD:SW_Push_SPST_NO_Alps_SKRK, symbol esp32-thing-eagle-import:SWITCH-MOMENTARY-2SMD-4.6X2.8MM
- added SW1: RESET, Button_Switch_SMD:SW_Push_SPST_NO_Alps_SKRK, symbol Switch:SW_Push
- added SW2: FLASH, Button_Switch_SMD:SW_Push_SPST_NO_Alps_SKRK, symbol Switch:SW_Push
Connections:
- net EN: now also SW1.2
- net GND: now also SW1.1, SW2.1; no longer J1.6 (Shield)
- net GPIO0: now also SW2.2
Changed lines of the file:
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@@
   (junction (at 186.69 58.42) (diameter 0) (color 0 0 0 0)
   )
+  (junction (at 180.34 67.31) (diameter 0) (color 0 0 0 0)
+  )
+  (junction (at 274.32 31.75) (diameter 0) (color 0 0 0 0)
+  )
   (junction (at 266.7 115.57) (diameter 0) (color 0 0 0 0)
   )
-  (junction (at 180.34 67.31) (diameter 0) (color 0 0 0 0)
-  )
-  (junction (at 274.32 31.75) (diameter 0) (color 0 0 0 0)
-  )
-  (junction (at 165.1 48.26) (diameter 0) (color 0 0 0 0)
-  )
   (junction (at 120.65 74.93) (diameter 0) (color 0 0 0 0)
   )
@@
     (stroke (width 0) (type default) (color 0 0 0 0))
   )
+  (wire (pts (xy 261.62 115.57) (xy 266.7 115.57))
+    (stroke (width 0) (type default) (color 0 0 0 0))
+  )
   (wire (pts (xy 246.38 25.4) (xy 246.38 31.75))
     (stroke (width 0) (type default) (color 0 0 0 0))
@@
     (stroke (width 0) (type default) (color 0 0 0 0))
   )
+  (wire (pts (xy 274.32 115.57) (xy 266.7 115.57))
+    (stroke (width 0) (type default) (color 0 0 0 0))
+  )
   (wire (pts (xy 207.01 116.84) (xy 207.01 119.38))
     (stroke (width 0) (type default) (color 0 0 0 0))
@@
     (stroke (width 0) (type default) (color 0 0 0 0))
   )
-  (wire (pts (xy 266.7 113.03) (xy 266.7 115.57))
-    (stroke (width 0) (type default) (color 0 0 0 0))
-  )
   (wire (pts (xy 274.32 27.94) (xy 274.32 31.75))
     (stroke (width 0) (type default) (color 0 0 0 0))
@@
     (stroke (width 0) (type default) (color 0 0 0 0))
   )
-  (wire (pts (xy 264.16 115.57) (xy 266.7 115.57))
-    (stroke (width 0) (type default) (color 0 0 0 0))
-  )
   (wire (pts (xy 246.38 31.75) (xy 252.73 31.75))
     (stroke (width 0) (type default) (color 0 0 0 0))
@@
     (stroke (width 0) (type default) (color 0 0 0 0))
   )
-  (wire (pts (xy 251.46 115.57) (xy 251.46 118.11))
+  (wire (pts (xy 246.38 115.57) (xy 246.38 118.11))
     (stroke (width 0) (type default) (color 0 0 0 0))
   )
@@
     (stroke (width 0) (type default) (color 0 0 0 0))
   )
-  (wire (pts (xy 254 115.57) (xy 251.46 115.57))
+  (wire (pts (xy 246.38 115.57) (xy 251.46 115.57))
     (stroke (width 0) (type default) (color 0 0 0 0))
   )
@@
     (stroke (width 0) (type default) (color 0 0 0 0))
   )
+  (wire (pts (xy 266.7 115.57) (xy 266.7 113.03))
+    (stroke (width 0) (type default) (color 0 0 0 0))
+  )
   (wire (pts (xy 255.27 78.74) (xy 257.81 78.74))
     (stroke (width 0) (type default) (color 0 0 0 0))
@@
     (stroke (width 0) (type default) (color 0 0 0 0))
   )
-  (wire (pts (xy 266.7 115.57) (xy 269.24 115.57))
-    (stroke (width 0) (type default) (color 0 0 0 0))
-  )
   (polyline (pts (xy 105.41 12.7) (xy 106.68 12.7))
     (stroke (width 0) (type default) (color 0 0 0 0))
@@
   )
   (polyline (pts (xy 229.87 12.7) (xy 229.87 85.09))
-    (stroke (width 0) (type default) (color 0 0 0 0))
-  )
-  (wire (pts (xy 162.56 48.26) (xy 165.1 48.26))
     (stroke (width 0) (type default) (color 0 0 0 0))
   )
@@
     (effects (font (size 1.27 1.27)) (justify right bottom))
   )
-  (label "EN" (at 269.24 115.57 0)
+  (label "EN" (at 274.32 115.57 0)
     (effects (font (size 0.889 0.889)) (justify left bottom))
   )
@@
     (pin "2")
   )
+  (symbol (lib_id "Switch:SW_Push") (at 256.54 115.57 0) (unit 1)
+    (in_bom yes) (on_board yes) (fields_autoplaced)
+    (property "Reference" "SW1" (id 0) (at 256.54 107.95 0))
+    (property "Value" "RESET" (id 1) (at 256.54 110.49 0))
+    (property "Footprint" "Button_Switch_SMD:SW_Push_SPST_NO_Alps_SKRK" (id 2) (at 256.54 110.49 0)
+      (effects (font (size 1.27 1.27)) hide)
+    )
+    (property "Datasheet" "~" (id 3) (at 256.54 110.49 0)
+      (effects (font (size 1.27 1.27)) hide)
+    )
+    (pin "1")
+    (pin "2")
+  )
   (symbol (lib_id "Device:Crystal_GND24") (at 180.34 58.42 0) (unit 1)
     (in_bom yes) (on_board yes) (fields_autoplaced)
@@
     (pin "4")
   )
-  (symbol (lib_id "esp32-thing-eagle-import:GND") (at 251.46 120.65 0) (unit 1)
+  (symbol (lib_id "esp32-thing-eagle-import:GND") (at 246.38 120.65 0) (unit 1)
     (in_bom yes) (on_board yes)
-    (property "Reference" "#GND0101" (id 0) (at 251.46 120.65 0)
-      (effects (font (size 1.27 1.27)) hide)
-    )
-    (property "Value" "GND" (id 1) (at 251.46 120.904 0)
+    (property "Reference" "#GND0101" (id 0) (at 246.38 120.65 0)
+      (effects (font (size 1.27 1.27)) hide)
+    )
+    (property "Value" "GND" (id 1) (at 246.38 120.904 0)
       (effects (font (size 1.778 1.5113)) (justify top))
     )
-    (property "Footprint" "esp32-thing:" (id 2) (at 251.46 120.65 0)
-      (effects (font (size 1.27 1.27)) hide)
-    )
-    (property "Datasheet" "" (id 3) (at 251.46 120.65 0)
+    (property "Footprint" "esp32-thing:" (id 2) (at 246.38 120.65 0)
+      (effects (font (size 1.27 1.27)) hide)
+    )
+    (property "Datasheet" "" (id 3) (at 246.38 120.65 0)
       (effects (font (size 1.27 1.27)) hide)
     )
@@
     (pin "1")
     (pin "2")
-  )
-  (symbol (lib_id "esp32-thing-eagle-import:SWITCH-MOMENTARY-2SMD-4.6X2.8MM") (at 214.63 116.84 0) (unit 1)
-    (in_bom yes) (on_board yes)
-    (property "Reference" "S2" (id 0) (at 212.09 114.3 0)
-      (effects (font (size 1.778 1.5113)) (justify left bottom))
-    )
-    (property "Value" "FLASH" (id 1) (at 212.09 120.65 0)
-      (effects (font (size 1.778 1.5113)) (justify left bottom))
-    )
-    (property "Footprint" "Button_Switch_SMD:SW_Push_SPST_NO_Alps_SKRK" (id 2) (at 214.63 116.84 0)
-      (effects (font (size 1.27 1.27)) hide)
-    )
-    (property "Datasheet" "" (id 3) (at 214.63 116.84 0)
-      (effects (font (size 1.27 1.27)) hide)
-    )
-    (pin "1")
-    (pin "2")
-    (pin "3")
-    (pin "4")
   )
   (symbol (lib_id "Device:C") (at 246.38 35.56 0) (unit 1)
@@
     (pin "2")
   )
-  (symbol (lib_id "esp32-thing-eagle-import:SWITCH-MOMENTARY-2SMD-4.6X2.8MM") (at 259.08 115.57 0) (unit 1)
-    (in_bom yes) (on_board yes)
-    (property "Reference" "S1" (id 0) (at 256.54 113.03 0)
-      (effects (font (size 1.778 1.5113)) (justify left bottom))
-    )
-    (property "Value" "RESET" (id 1) (at 256.54 119.38 0)
-      (effects (font (size 1.778 1.5113)) (justify left bottom))
-    )
-    (property "Footprint" "Button_Switch_SMD:SW_Push_SPST_NO_Alps_SKRK" (id 2) (at 259.08 115.57 0)
-      (effects (font (size 1.27 1.27)) hide)
-    )
-    (property "Datasheet" "" (id 3) (at 259.08 115.57 0)
-      (effects (font (size 1.27 1.27)) hide)
-    )
-    (pin "1")
-    (pin "2")
-    (pin "3")
-    (pin "4")
-  )
   (symbol (lib_id "Device:C") (at 186.69 27.94 0) (unit 1)
     (in_bom yes) (on_board yes)
@@
     (pin "6")
   )
+  (symbol (lib_id "Switch:SW_Push") (at 214.63 116.84 0) (unit 1)
+    (in_bom yes) (on_board yes) (fields_autoplaced)
+    (property "Reference" "SW2" (id 0) (at 214.63 109.22 0))
+    (property "Value" "FLASH" (id 1) (at 214.63 111.76 0))
+    (property "Footprint" "Button_Switch_SMD:SW_Push_SPST_NO_Alps_SKRK" (id 2) (at 214.63 111.76 0)
+      (effects (font (size 1.27 1.27)) hide)
+    )
+    (property "Datasheet" "~" (id 3) (at 214.63 111.76 0)
+      (effects (font (size 1.27 1.27)) hide)
+    )
+    (pin "1")
+    (pin "2")
+  )
   (symbol (lib_id "Device:D_Schottky") (at 189.23 20.32 180) (unit 1)
     (in_bom yes) (on_board yes) (fields_autoplaced)
@@
   (symbol (lib_id "esp32-thing-eagle-import:3.3V") (at 274.32 27.94 0) (unit 1)
     (in_bom yes) (on_board yes)
-    (property "Reference" "#SUPPLY?" (id 0) (at 274.32 27.94 0)
+    (property "Reference" "#SUPPLY0103" (id 0) (at 274.32 27.94 0)
       (effects (font (size 1.27 1.27)) hide)
     )
@@
     )
     (path "/f5a93514-35cd-4204-84c8-cda248428de4"
-      (reference "#SUPPLY?") (unit 1) (value "+3.3V") (footprint "esp32-thing:")
+      (reference "#SUPPLY0103") (unit 1) (value "+3.3V") (footprint "esp32-thing:")
     )
     (path "/721477dc-631a-4178-857f-787efd54dcc9"
@@
       (reference "R6") (unit 1) (value "10k") (footprint "Resistor_SMD:R_0805_2012Metric_Pad1.20x1.40mm_HandSolder")
     )
-    (path "/ae5892e8-b97b-49ae-93a5-c4a8909413ff"
-      (reference "S1") (unit 1) (value "RESET") (footprint "Button_Switch_SMD:SW_Push_SPST_NO_Alps_SKRK")
-    )
-    (path "/77283ea7-277d-49f5-9f10-d65edc4b3e49"
-      (reference "S2") (unit 1) (value "FLASH") (footprint "Button_Switch_SMD:SW_Push_SPST_NO_Alps_SKRK")
+    (path "/0b8f40fb-1eb3-47e8-a630-bb3a7e9d4bb9"
+      (reference "SW1") (unit 1) (value "RESET") (footprint "Button_Switch_SMD:SW_Push_SPST_NO_Alps_SKRK")
+    )
+    (path "/cb9bc265-fb15-4997-9d96-28c657561798"
+      (reference "SW2") (unit 1) (value "FLASH") (footprint "Button_Switch_SMD:SW_Push_SPST_NO_Alps_SKRK")
     )
     (path "/90251756-a362-493b-b950-73ddaf1c8246"
